File: hardware/Ideal OR Diode.kicad_sch (KiCad schematic)
At the start: 18 parts, among them J1 PWR A, J2 PWR B, J3 PWR OUT, J4 Conn_01x03_Pin, Q1 BSC030N03LS_G, Q2 BSC030N03LS_G, Q3 BSC030N03LS_G, Q4 BSC030N02LS_G, U1 LTC4353IMS

Commit message: Update the Sheet frames to show URL
Other:
- company: (none) -> VA7DBI
- title: (none) -> Ideal OR Diode
Changed lines of the file:
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@@
 	(generator "eeschema")
 	(generator_version "8.0")
-	(paper "A4")
+	(paper "USLetter")
+	(title_block
+		(title "Ideal OR Diode")
+		(date "2024-04-11")
+		(rev "1.0")
+		(company "VA7DBI")
+		(comment 1 "http://github.com/VA7DBI/ideal-or-diode")
+	)
 	(junction
 		(at 130.81 67.31)
